File: Balance_Bot.kicad_pcb (KiCad board)
At the start: 4 copper layers, 78 x 60 mm, 57 parts, among them CN1 Battery Power, J10 DRV8825_1_M2, J11 Conn_01x10, J12 Left, J13 Right, J14 Conn_01x16, J5 DRV8825_0_M0, J6 DRV8825_0_M1, J7 DRV8825_0_M2, J8 DRV8825_1_M0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

Commit message: Github Prep (#1)
Prepping repo to be published onto public GitHub.  Made general corrections, wrote a README, and tidied up the repo.

Co-authored-by: TheFlemoid <trey.dahlberg@gmail.com>
Reviewed-on: https://git.tdberg.com/TheFlemoid/ESP-32-Stepper-Driver/pulls/1
Parts:
- renumbered SW2 to BOOT, SW1 to RESET
Other:
- board text added: "JLCJLCJLCJLC"
